File: ina-connector.kicad/ina-connector.kicad_pcb (KiCad board)
At the start: 2 copper layers, 21 x 68 mm, 13 parts, among them J1 Vin JST-PH2, J2 Vin Header*, J3 Vin Barrel-Jack, J4 Vout AKL, J5 Vout Header*, J6 Conn_INA, J7 GND, J8 GND, SW1 SW_SPST

Commit message: Rev. 1.10: use thermal reliefs
Other:
- board text added: "Rev: 1.10"
- board text removed: "Rev: 1.00"
Changed lines of the file:
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@@
     (effects (font (size 1 1) (thickness 0.15)) (justify left bottom mirror))
   )
-  (gr_text "Rev: 1.00" (at 101.69825 104.7 90) (layer "B.SilkS")
+  (gr_text "Rev: 1.10" (at 101.69825 104.7 90) (layer "B.SilkS")
     (effects (font (size 1 1) (thickness 0.15)) (justify left mirror))
   )
@@
   (zone (net 2) (net_name "Net-(J1-Pin_1)") (layer "F.Cu") (hatch edge 0.5)
     (priority 4)
-    (connect_pads yes (clearance 0.508))
+    (connect_pads (clearance 0.508))
     (min_thickness 0.25) (filled_areas_thickness no)
     (fill yes (thermal_gap 0.5) (thermal_bridge_width 0.5))
@@
   (zone (net 4) (net_name "Net-(J6-Pin_1)") (layer "F.Cu") (hatch edge 0.5)
     (priority 4)
-    (connect_pads yes (clearance 0.508))
+    (connect_pads (clearance 0.508))
     (min_thickness 0.25) (filled_areas_thickness no)
     (fill yes (thermal_gap 0.5) (thermal_bridge_width 0.5))
@@
   (zone (net 3) (net_name "Net-(J4-Pin_1)") (layer "F.Cu") (hatch edge 0.5)
     (priority 4)
-    (connect_pads yes (clearance 0.508))
+    (connect_pads (clearance 0.508))
     (min_thickness 0.25) (filled_areas_thickness no)
     (fill yes (thermal_gap 0.5) (thermal_bridge_width 0.5))
@@
   (zone (net 1) (net_name "GND") (layers "F&B.Cu") (hatch edge 0.5)
     (priority 2)
-    (connect_pads yes (clearance 0.508))
+    (connect_pads (clearance 0.508))
     (min_thickness 0.25) (filled_areas_thickness no)
     (fill yes (thermal_gap 0.5) (thermal_bridge_width 0.5))
